File: pcb/eagle/adc_microboard.brd (EAGLE design)
At the start: 45.5 x 41.9 mm, 93 parts, among them T1 TC1-1T, U1 AD9215BRUZ, U2 AD8331, U3 LP3985IM5-3.0, U4 LTC3200ES6, X1 SMA-142-0711-821/826, X2 SMA-142-0711-821/826, X3 BU-SMA-V

Commit message: Add mounting holes, update silkscreen
Parts:
- added H1: MOUNT-PAD-ROUND2.8, holes:2,8-PAD
- moved C37 0.20 mm to (31.3, 3.41)
- moved C46 0.10 mm to (31.3, 4.30)
Connections:
- net AGND: now also H1.B2,8
Routing:
- net N$35: track 38.1 -> 38.6 mm
Other:
- board text removed: "1.65""
- board text removed: "1.79""
- board text removed: "IN-AMP"
- board text removed: "IN-XFRMER"
