File: pcb/eagle/adc_microboard.brd (EAGLE design)
At the start: 45.5 x 41.9 mm, 94 parts, among them T1 TC1-1T, U1 AD9215BRUZ, U2 AD8331, U3 LP3985IM5-3.0, U4 LTC3200ES6, X1 SMA-142-0711-821/826, X2 SMA-142-0711-821/826, X3 BU-SMA-V

Commit message: Update PCB to include fixes
Parts:
- added C48: 22pF, rcl:C0603
- moved H1 0.33 mm to (12.9, 21.5)
Connections:
- net AGND: now also C48.2
- net N$16: now also C48.1
Routing:
- net N$16: track 4.13 -> 5.67 mm
- net AGND: vias 79 -> 80
Other:
- board text added: "1"
- board text added: "ADC0"
- board text added: "ADC1"
- board text added: "ADC2"
- board text added: "ADC3"
- board text added: "ADC4"
- board text added: "ADC5"
- board text added: "ADC6"
- board text added: "ADC7"
- board text added: "ADC8"
- board text added: "ADC9"
- board text added: "ADC_OR"
- board text added: "GAINMODE"
- board text added: "TRIGGER"
- board text added: "VCC"
