File: pcb/eagle/adc_microboard.brd (EAGLE design)
At the start: 45.5 x 41.9 mm, 95 parts, among them T1 TC1-1T, U1 AD9215BRUZ, U2 AD8331, U3 LP3985IM5-3.0, U4 LTC3200ES6, X1 SMA-142-0711-821/826, X2 SMA-142-0711-821/826, X3 BU-SMA-V

Commit message: Update PCB
Parts:
- C47: value 1nF -> 1uF
- R14: device adafruit:R0402 -> adafruit:R0603
- R9: value (none) -> 390R
- moved R14 0.13 mm to (36.1, 17.3)
Other:
- board text added: "Pb-Free"
- board text added: "Revision 28AUG2012"
- board text added: "RoHS"
- board text added: "S/N:"
Changed lines of the file:
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@@
 <layer number="15" name="Route15" color="4" fill="6" visible="no" active="no"/>
 <layer number="16" name="Bottom" color="1" fill="1" visible="yes" active="yes"/>
-<layer number="17" name="Pads" color="2" fill="1" visible="no" active="yes"/>
-<layer number="18" name="Vias" color="2" fill="1" visible="no" active="yes"/>
+<layer number="17" name="Pads" color="2" fill="1" visible="yes" active="yes"/>
+<layer number="18" name="Vias" color="2" fill="1" visible="yes" active="yes"/>
 <layer number="19" name="Unrouted" color="6" fill="1" visible="no" active="yes"/>
-<layer number="20" name="Dimension" color="15" fill="1" visible="no" active="yes"/>
-<layer number="21" name="tPlace" color="7" fill="1" visible="no" active="yes"/>
+<layer number="20" name="Dimension" color="15" fill="1" visible="yes" active="yes"/>
+<layer number="21" name="tPlace" color="7" fill="1" visible="yes" active="yes"/>
 <layer number="22" name="bPlace" color="7" fill="1" visible="yes" active="yes"/>
-<layer number="23" name="tOrigins" color="15" fill="1" visible="no" active="yes"/>
+<layer number="23" name="tOrigins" color="15" fill="1" visible="yes" active="yes"/>
 <layer number="24" name="bOrigins" color="15" fill="1" visible="no" active="yes"/>
 <layer number="25" name="tNames" color="7" fill="1" visible="no" active="yes"/>
@@
 <layer number="49" name="Reference" color="7" fill="1" visible="no" active="yes"/>
 <layer number="50" name="dxf" color="7" fill="1" visible="no" active="yes"/>
-<layer number="51" name="tDocu" color="7" fill="1" visible="no" active="yes"/>
+<layer number="51" name="tDocu" color="7" fill="1" visible="yes" active="yes"/>
 <layer number="52" name="bDocu" color="7" fill="1" visible="no" active="yes"/>
 <layer number="53" name="tGND_GNDA" color="7" fill="9" visible="no" active="no"/>
@@
 <layer number="213" name="213bmp" color="7" fill="1" visible="no" active="yes"/>
 <layer number="214" name="214bmp" color="7" fill="1" visible="no" active="yes"/>
-<layer number="215" name="bottomopenadc" color="15" fill="1" visible="yes" active="yes"/>
+<layer number="215" name="bottomopenadc" color="15" fill="1" visible="no" active="yes"/>
 <layer number="216" name="216bmp" color="1" fill="10" visible="no" active="yes"/>
 <layer number="217" name="217bmp" color="18" fill="1" visible="no" active="no"/>
@@
 <layer number="220" name="220bmp" color="21" fill="1" visible="no" active="no"/>
 <layer number="221" name="221bmp" color="22" fill="1" visible="no" active="no"/>
-<layer number="222" name="222bmp" color="23" fill="1" visible="no" active="no"/>
 <layer number="223" name="223bmp" color="24" fill="1" visible="no" active="no"/>
 <layer number="224" name="224bmp" color="25" fill="1" visible="no" active="no"/>
@@
 <rectangle x1="39.106334375" y1="8.346490625" x2="39.686234375" y2="8.378696875" layer="215" rot="R309.4"/>
 <text x="31.084578125" y="3.1889875" size="1.6764" layer="22" font="vector" ratio="16" rot="MR51">www.newae.com/openadc</text>
-<text x="34.853384375" y="34.98223125" size="1.27" layer="22" font="vector" ratio="16" rot="MR0">3.3V Only</text>
+<text x="40.2972125" y="31.02015625" size="1.27" layer="22" font="vector" ratio="16" rot="MR270">3.3V Only</text>
+<text x="28.2821375" y="3.060140625" size="1.016" layer="22" font="vector" ratio="16" rot="MR0">Revision 28AUG2012</text>
+<text x="28.2821375" y="4.50968125" size="1.016" layer="22" font="vector" ratio="16" rot="MR0">Pb-Free</text>
+<text x="20.390196875" y="4.44525625" size="1.016" layer="22" font="vector" ratio="16" rot="MR0">RoHS</text>
+<text x="27.444625" y="6.12028125" size="1.016" layer="22" font="vector" ratio="16" rot="MR0">S/N:</text>
+<rectangle x1="10.340053125" y1="5.95921875" x2="23.933515625" y2="8.0207875" layer="22"/>
 </plain>
 <attributes>
@@
 <attribute name="PART#" value="GRM155R61A104KA01D" x="27.305" y="6.9749" size="1.778" layer="27" rot="R270" display="off"/>
 </element>
-<element name="R9" library="adafruit" package="R0603" value="" x="28.8874" y="6.9749" smashed="yes" rot="R270">
+<element name="R9" library="adafruit" package="R0603" value="390R" x="28.8874" y="6.9749" smashed="yes" rot="R270">
 <attribute name="NAME" x="28.4379" y="5.7303" size="1.016" layer="25" font="vector" ratio="16" rot="R270"/>
 <attribute name="VALUE" x="26.8554" y="7.8639" size="1.27" layer="27" rot="R270"/>
@@
 <attribute name="VALUE" x="30.292" y="22.2682" size="1.27" layer="27" rot="R90"/>
 </element>
-<element name="R14" library="adafruit" package="R0402" value="" x="36.1289" y="17.4193" smashed="yes" rot="R180">
-<attribute name="NAME" x="35.2316" y="17.7863" size="1.016" layer="25" font="vector" ratio="16" rot="R180"/>
-<attribute name="VALUE" x="36.7639" y="19.4513" size="1.27" layer="27" rot="R180"/>
+<element name="R14" library="adafruit" package="R0603" value="" x="36.1289" y="17.29045" smashed="yes" rot="R180">
+<attribute name="NAME" x="35.2316" y="17.65745" size="1.016" layer="25" font="vector" ratio="16" rot="R180"/>
+<attribute name="VALUE" x="36.7639" y="19.32245" size="1.27" layer="27" rot="R180"/>
 </element>
 <element name="R13" library="customs" package="3361P" value="20k" x="26.1288" y="30.6451" smashed="yes">
@@
 <attribute name="VALUE" x="31.935" y="6.2034" size="1.27" layer="27" rot="R180"/>
 </element>
-<element name="C47" library="rcl" package="C0402" value="1nF" x="29.1" y="10.9" smashed="yes" rot="R90">
+<element name="C47" library="rcl" package="C0402" value="1uF" x="29.1" y="10.9" smashed="yes" rot="R90">
 <attribute name="DIGIKEY#" value="445-4924-1-ND" x="29.1" y="10.9" size="1.778" layer="27" rot="R90" display="off"/>
 <attribute name="PART#" value="C1005X7R1E102K" x="29.1" y="10.9" size="1.778" layer="27" rot="R90" display="off"/>
@@
 <wire x1="42.903" y1="23.8661" x2="43.96" y2="24.408" width="0.4" layer="1" curve="54.286384"/>
 <via x="43.96" y="24.408" extent="1-16" drill="0.4318"/>
-<wire x1="36.7789" y1="17.4193" x2="36.744" y2="18.904" width="0.4" layer="1"/>
+<wire x1="36.9789" y1="17.29045" x2="36.744" y2="18.904" width="0.4" layer="1"/>
 <via x="36.744" y="18.904" extent="1-16" drill="0.4318"/>
 <via x="36.528" y="21.728" extent="1-16" drill="0.4318"/>
@@
 <wire x1="37.4574" y1="14.8006" x2="39.558" y2="12.7" width="0.381" layer="1"/>
 <wire x1="35.4838" y1="17.4144" x2="35.4838" y2="16.7742" width="0.381" layer="1"/>
-<wire x1="35.4789" y1="17.4193" x2="35.4838" y2="17.4144" width="0.381" layer="1"/>
-<wire x1="35.4789" y1="17.4193" x2="35.4789" y2="17.7468" width="0.381" layer="1"/>
+<wire x1="35.2789" y1="17.29045" x2="35.4838" y2="17.4144" width="0.381" layer="1"/>
+<wire x1="35.2789" y1="17.29045" x2="35.4789" y2="17.7468" width="0.381" layer="1"/>
 <wire x1="35.4789" y1="17.7468" x2="35.1612" y2="18.0645" width="0.381" layer="1"/>
 <via x="37.084" y="15.24" extent="1-16" drill="0.9" shape="octagon"/>

Commit message: Update PCB
Parts:
- added C49: (no value), adc_microboard:C0603
- added D1, D2, D3: BAV99-7-F, zetex:SOT-23
- R19: device adafruit:R0603 -> adafruit:R0805
- R9: value 390R -> 10K
- moved C39 1.66 mm to (16.5, 7.34), turned to 180 degrees
- moved R16 1.39 mm to (17.4, 4.42)
Connections:
- net +3V3: now also C49.1, D1.2, D2.2
- net AGND: now also C49.2, D1.3, D2.3, D3.2
- net N$18: now also D2.1
- net N$37: now also D3.3
- net N$44: now also D1.1
Routing:
- net N$44: track 27.0 -> 45.9 mm
- net +3V3: track 28.7 -> 46.7 mm
- net N$37: track 3.51 -> 7.01 mm
- net ADC_OR: track 24.7 -> 27.1 mm
- net ADC8: track 19.9 -> 17.9 mm
- net ADC6: track 18.3 -> 16.6 mm
- net ADC7: track 15.8 -> 14.2 mm
- net ADC9: track 17.3 -> 15.8 mm
- net N$36: track 42.5 -> 41.1 mm
- net N$18: track 20.1 -> 20.7 mm
- net AGND: track 86.6 -> 87.1 mm
Other:
- board text added: "CLOCK_IN"
- board text added: "GAIN"
- board text added: "Revision 28NOV2012"
- board text added: "TRIGGER_IN"
- board text removed: "C:/E/Documents/openadc/newae.com.bmp"
- board text removed: "Revision 28AUG2012"
- board text removed: "TRIGGER"
