File: pcb/eagle/adc_microboard.sch (EAGLE design)
At the start: 95 parts, among them T1 TC1-1T, U1 AD9215BRUZ, U2 AD8331, U3 LP3985IM5-3.0, U4 LTC3200ES6, X1 SMA-142-0711-821/826, X2 SMA-142-0711-821/826, X3 BU-SMA-V

Commit message: Update PCB
Parts:
- added C49: (no value), adc_microboard:C-EUC0603
- added D1, D2, D3: BAV99-7-F, zetex:D_ACACSOT23
- R19: device adafruit:R-US_R0603 -> adafruit:R-US_R0805
- R9: value 390R -> 10K
Connections:
- net +3V3: now also C49.1, D1.C, D2.C
- net AGND: now also C49.2, D1.A, D2.A, D3.C
- net N$18: now also D2.CA
- net N$37: now also D3.A
- net N$44: now also D1.CA
Changed lines of the file:
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@@
 <?xml version="1.0" encoding="utf-8"?>
 <!DOCTYPE eagle SYSTEM "eagle.dtd">
-<eagle version="6.2">
+<eagle version="6.3">
 <drawing>
 <settings>
@@
 <layer number="250" name="Descript" color="7" fill="1" visible="no" active="no"/>
 <layer number="251" name="SMDround" color="7" fill="1" visible="no" active="no"/>
+<layer number="253" name="NotesToFab" color="7" fill="1" visible="yes" active="yes"/>
 <layer number="254" name="cooling" color="7" fill="1" visible="yes" active="yes"/>
 </layers>
@@
 <part name="SUPPLY6" library="supply2" deviceset="AGND" device=""/>
 <part name="SUPPLY7" library="supply2" deviceset="AGND" device=""/>
-<part name="R9" library="adafruit" deviceset="R-US_" device="R0603" value="390R"/>
+<part name="R9" library="adafruit" deviceset="R-US_" device="R0603" value="10K"/>
 <part name="SUPPLY8" library="supply2" deviceset="AGND" device=""/>
 <part name="C9" library="rcl" deviceset="C-EU" device="C0402" value="100nF">
@@
 <part name="+3V2" library="supply1" deviceset="+3V3" device=""/>
 <part name="X3" library="con-coax" deviceset="BU-SMA-V" device=""/>
-<part name="R19" library="adafruit" deviceset="R-US_" device="R0603"/>
+<part name="R19" library="adafruit" deviceset="R-US_" device="R0805"/>
 <part name="JP9" library="pinhead" deviceset="PINHD-1X2" device="/90">
 <attribute name="DIGIKEY#" value="WM2711-ND"/>
@@
 </part>
 <part name="SUPPLY55" library="supply2" deviceset="AGND" device=""/>
+<part name="D1" library="zetex" deviceset="D_ACAC" device="SOT23" value="BAV99-7-F"/>
+<part name="D2" library="zetex" deviceset="D_ACAC" device="SOT23" value="BAV99-7-F"/>
+<part name="+3V6" library="supply1" deviceset="+3V3" device=""/>
+<part name="C49" library="adc_microboard" deviceset="C-EU" device="C0603"/>
+<part name="SUPPLY56" library="supply2" deviceset="AGND" device=""/>
+<part name="D3" library="zetex" deviceset="D_ACAC" device="SOT23" value="BAV99-7-F"/>
+<part name="SUPPLY57" library="supply2" deviceset="AGND" device=""/>
 </parts>
 <sheets>
@@
 </instance>
 <instance part="SUPPLY55" gate="G$1" x="27.94" y="40.64" rot="R270"/>
+<instance part="D3" gate="A" x="127" y="20.32"/>
+<instance part="SUPPLY57" gate="G$1" x="124.46" y="15.24"/>
 </instances>
 <busses>
@@
 <pinref part="C48" gate="G$1" pin="2"/>
 <pinref part="SUPPLY55" gate="G$1" pin="AGND"/>
+</segment>
+<segment>
+<pinref part="D3" gate="A" pin="C"/>
+<pinref part="SUPPLY57" gate="G$1" pin="AGND"/>
 </segment>
 </net>
@@
 <pinref part="C39" gate="G$1" pin="1"/>
 <pinref part="U2" gate="G$1" pin="GAIN"/>
+<pinref part="D3" gate="A" pin="A"/>
+<wire x1="124.46" y1="22.86" x2="124.46" y2="40.64" width="0.1524" layer="91"/>
+<junction x="124.46" y="40.64"/>
 </segment>
 </net>
@@
 <instance part="H1" gate="G$1" x="50.8" y="66.04"/>
 <instance part="SUPPLY54" gate="G$1" x="43.18" y="60.96"/>
+<instance part="D1" gate="A" x="132.08" y="154.94" rot="R90"/>
+<instance part="D2" gate="A" x="132.08" y="147.32" rot="MR270"/>
+<instance part="+3V6" gate="G$1" x="165.1" y="152.4" rot="R270"/>
+<instance part="C49" gate="G$1" x="152.4" y="147.32" rot="R90"/>
+<instance part="SUPPLY56" gate="G$1" x="160.02" y="147.32" rot="R90"/>
 </instances>
 <busses>
@@
 <pinref part="JP2" gate="A" pin="11"/>
 </segment>
+<segment>
+<pinref part="D2" gate="A" pin="C"/>
+<pinref part="D1" gate="A" pin="C"/>
+<wire x1="134.62" y1="149.86" x2="134.62" y2="152.4" width="0.1524" layer="91"/>
+<pinref part="+3V6" gate="G$1" pin="+3V3"/>
+<wire x1="162.56" y1="152.4" x2="144.78" y2="152.4" width="0.1524" layer="91"/>
+<junction x="134.62" y="152.4"/>
+<pinref part="C49" gate="G$1" pin="1"/>
+<wire x1="144.78" y1="152.4" x2="134.62" y2="152.4" width="0.1524" layer="91"/>
+<wire x1="149.86" y1="147.32" x2="144.78" y2="147.32" width="0.1524" layer="91"/>
+<wire x1="144.78" y1="147.32" x2="144.78" y2="152.4" width="0.1524" layer="91"/>
+<junction x="144.78" y="152.4"/>
+</segment>
 </net>
 <net name="ADC_OR" class="0">
@@
 <net name="N$18" class="0">
 <segment>
-<wire x1="111.76" y1="142.24" x2="167.64" y2="142.24" width="0.1524" layer="91"/>
+<wire x1="111.76" y1="142.24" x2="132.08" y2="142.24" width="0.1524" layer="91"/>
+<wire x1="132.08" y1="142.24" x2="167.64" y2="142.24" width="0.1524" layer="91"/>
 <wire x1="167.64" y1="142.24" x2="167.64" y2="139.7" width="0.1524" layer="91"/>
 <wire x1="167.64" y1="139.7" x2="180.34" y2="139.7" width="0.1524" layer="91"/>
 <pinref part="R19" gate="G$1" pin="2"/>
 <pinref part="JP1" gate="A" pin="1"/>
+<pinref part="D2" gate="A" pin="CA"/>
+<junction x="132.08" y="142.24"/>
 </segment>
 </net>
@@
 <net name="N$44" class="0">
 <segment>
-<wire x1="114.3" y1="160.02" x2="193.04" y2="160.02" width="0.1524" layer="91"/>
+<wire x1="114.3" y1="160.02" x2="132.08" y2="160.02" width="0.1524" layer="91"/>
+<wire x1="132.08" y1="160.02" x2="193.04" y2="160.02" width="0.1524" layer="91"/>
 <wire x1="193.04" y1="160.02" x2="193.04" y2="139.7" width="0.1524" layer="91"/>
 <wire x1="193.04" y1="139.7" x2="187.96" y2="139.7" width="0.1524" layer="91"/>
 <pinref part="R21" gate="G$1" pin="2"/>
 <pinref part="JP1" gate="A" pin="2"/>
+<pinref part="D1" gate="A" pin="CA"/>
+<junction x="132.08" y="160.02"/>
 </segment>
 </net>
@@
 <pinref part="R20" gate="G$1" pin="2"/>
 <pinref part="SUPPLY51" gate="G$1" pin="AGND"/>
+<pinref part="D2" gate="A" pin="A"/>
+<pinref part="D1" gate="A" pin="A"/>
+<wire x1="129.54" y1="149.86" x2="129.54" y2="152.4" width="0.1524" layer="91"/>
+<wire x1="129.54" y1="149.86" x2="116.84" y2="149.86" width="0.1524" layer="91"/>
+<wire x1="116.84" y1="149.86" x2="116.84" y2="157.48" width="0.1524" layer="91"/>
+<junction x="129.54" y="149.86"/>
+<wire x1="116.84" y1="157.48" x2="109.22" y2="157.48" width="0.1524" layer="91"/>
+<junction x="109.22" y="157.48"/>
 </segment>
 <segment>
@@
 <wire x1="48.26" y1="66.04" x2="43.18" y2="66.04" width="0.1524" layer="91"/>
 </segment>
-</net>
+<segment>
+<pinref part="SUPPLY56" gate="G$1" pin="AGND"/>
+<pinref part="C49" gate="G$1" pin="2"/>
+</segment>
+</net>
